File: Traszka/Traszka.sch (EAGLE design)
At the start: 12 parts, among them IC1 MEGA8-P, IC2 7818TV, X3 CRYSTALS-NOGND-HC49

Commit message: Final version
Parts:
- added C5: (no value), rcl:C-EU050-024X044
- added R1, R2, R4: (no value), rcl:R-EU_0204/7
- added R3: (no value), rcl:R-EU_0204/5
- added T1: BC547, transistor:BC547
Connections:
- new net CHECK_VIN: IC1.PC4(ADC4/SDA), R4.1
- new net N$1: IC1.PC6(/RESET), R1.2
- new net N$2: C5.1, IC1.AREF
- new net N$3: R4.2, T1.B
- new net N$4: R3.1, T1.C
- new net VCCREF: IC1.PC0(ADC0), R2.1, R3.2
- net +5V: now also R1.1
- net +9V: now also R2.2
- net GND: now also C5.2, IC1.GND, T1.E
Other:
- moved on the sheet: C1, C2, C3, C4, IC1, IC2, SV1, SV2, SV3, SV4, X1-1, X1-2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

Commit message: fixing .sch and .brd checking battery
Connections:
- removed net N$4 (its old number): R3.1, T1.C
- new net N$3: R2.1, T1.C
- net GND: now also R3.1; no longer T1.E
- net VCCREF: now also T1.E; no longer R2.1
Other:
- moved on the sheet: R3, R4, T1
Changed lines of the file:
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@@
 <part name="C5" library="rcl" library_urn="urn:adsk.eagle:library:334" deviceset="C-EU" device="050-024X044" package3d_urn="urn:adsk.eagle:package:23643/1"/>
 <part name="GND11" library="supply1" library_urn="urn:adsk.eagle:library:371" deviceset="GND" device=""/>
-<part name="T1" library="transistor" library_urn="urn:adsk.eagle:library:402" deviceset="BC547" device="" package3d_urn="urn:adsk.eagle:package:28523/2"/>
 <part name="GND12" library="supply1" library_urn="urn:adsk.eagle:library:371" deviceset="GND" device=""/>
 <part name="SUPPLY10" library="supply2" library_urn="urn:adsk.eagle:library:372" deviceset="+9V" device=""/>
 <part name="R4" library="rcl" library_urn="urn:adsk.eagle:library:334" deviceset="R-EU_" device="0204/7" package3d_urn="urn:adsk.eagle:package:23498/2"/>
+<part name="T1" library="transistor" library_urn="urn:adsk.eagle:library:402" deviceset="BC547" device="" package3d_urn="urn:adsk.eagle:package:28523/2"/>
 </parts>
 <sheets>
@@
 <attribute name="VALUE" x="-14.478" y="46.99" size="1.778" layer="96" rot="R90"/>
 </instance>
-<instance part="R3" gate="G$1" x="-17.78" y="38.1" smashed="yes" rot="R90" grouprefs="BATTERY_CHECK">
-<attribute name="NAME" x="-19.2786" y="34.29" size="1.778" layer="95" rot="R90"/>
-<attribute name="VALUE" x="-14.478" y="34.29" size="1.778" layer="96" rot="R90"/>
+<instance part="R3" gate="G$1" x="-17.78" y="25.4" smashed="yes" rot="R90" grouprefs="BATTERY_CHECK">
+<attribute name="NAME" x="-19.2786" y="21.59" size="1.778" layer="95" rot="R90"/>
+<attribute name="VALUE" x="-14.478" y="21.59" size="1.778" layer="96" rot="R90"/>
 </instance>
 <instance part="C5" gate="G$1" x="71.12" y="50.8" smashed="yes" rot="R270" grouprefs="ARDUINO">
@@
 <attribute name="VALUE" x="63.5" y="43.18" size="1.778" layer="96"/>
 </instance>
-<instance part="T1" gate="G$1" x="-20.32" y="27.94" smashed="yes" grouprefs="BATTERY_CHECK">
-<attribute name="NAME" x="-30.48" y="35.56" size="1.778" layer="95"/>
-<attribute name="VALUE" x="-30.48" y="33.02" size="1.778" layer="96"/>
-</instance>
 <instance part="GND12" gate="1" x="-17.78" y="17.78" smashed="yes" grouprefs="BATTERY_CHECK">
 <attribute name="VALUE" x="-20.32" y="15.24" size="1.778" layer="96"/>
@@
 <attribute name="VALUE" x="-19.685" y="61.595" size="1.778" layer="96"/>
 </instance>
-<instance part="R4" gate="G$1" x="-27.94" y="27.94" smashed="yes" grouprefs="BATTERY_CHECK">
-<attribute name="NAME" x="-31.75" y="29.4386" size="1.778" layer="95"/>
-<attribute name="VALUE" x="-31.75" y="24.638" size="1.778" layer="96"/>
+<instance part="R4" gate="G$1" x="-27.94" y="38.1" smashed="yes" grouprefs="BATTERY_CHECK">
+<attribute name="NAME" x="-31.75" y="39.5986" size="1.778" layer="95"/>
+<attribute name="VALUE" x="-31.75" y="34.798" size="1.778" layer="96"/>
+</instance>
+<instance part="T1" gate="G$1" x="-20.32" y="38.1" smashed="yes" grouprefs="BATTERY_CHECK">
+<attribute name="NAME" x="-30.48" y="45.72" size="1.778" layer="95"/>
+<attribute name="VALUE" x="-30.48" y="43.18" size="1.778" layer="96"/>
 </instance>
 </instances>
@@
 <segment>
 <pinref part="GND12" gate="1" pin="GND"/>
-<pinref part="T1" gate="G$1" pin="E"/>
-<wire x1="-17.78" y1="20.32" x2="-17.78" y2="22.86" width="0.1524" layer="91" grouprefs="BATTERY_CHECK"/>
+<pinref part="R3" gate="G$1" pin="1"/>
 </segment>
 </net>
@@
 <net name="VCCREF" class="0">
 <segment>
-<pinref part="R2" gate="G$1" pin="1"/>
-<pinref part="R3" gate="G$1" pin="2"/>
-<label x="-17.78" y="45.72" size="1.778" layer="95" xref="yes" grouprefs="BATTERY_CHECK"/>
-<wire x1="-17.78" y1="45.72" x2="-17.78" y2="43.18" width="0.1524" layer="91" grouprefs="BATTERY_CHECK"/>
-</segment>
-<segment>
 <pinref part="IC1" gate="G$1" pin="PC0(ADC0)"/>
 <wire x1="124.46" y1="60.96" x2="127" y2="60.96" width="0.1524" layer="91" grouprefs="ARDUINO"/>
 <label x="127" y="60.96" size="1.778" layer="95" xref="yes" grouprefs="ARDUINO"/>
 </segment>
+<segment>
+<pinref part="R3" gate="G$1" pin="2"/>
+<pinref part="T1" gate="G$1" pin="E"/>
+<wire x1="-17.78" y1="30.48" x2="-17.78" y2="33.02" width="0.1524" layer="91" grouprefs="BATTERY_CHECK"/>
+<label x="-17.78" y="33.02" size="1.778" layer="95" xref="yes" grouprefs="BATTERY_CHECK"/>
+</segment>
 </net>
 <net name="N$2" class="0">
@@
 </segment>
 </net>
-<net name="N$4" class="0">
-<segment>
-<pinref part="R3" gate="G$1" pin="1"/>
-<pinref part="T1" gate="G$1" pin="C"/>
-</segment>
-</net>
 <net name="CHECK_VIN" class="0">
 <segment>
-<label x="-35.56" y="27.94" size="1.778" layer="95" rot="R90" xref="yes" grouprefs="BATTERY_CHECK"/>
-<wire x1="-33.02" y1="27.94" x2="-35.56" y2="27.94" width="0.1524" layer="91" grouprefs="BATTERY_CHECK"/>
+<label x="-35.56" y="38.1" size="1.778" layer="95" rot="R90" xref="yes" grouprefs="BATTERY_CHECK"/>
+<wire x1="-33.02" y1="38.1" x2="-35.56" y2="38.1" width="0.1524" layer="91" grouprefs="BATTERY_CHECK"/>
 <pinref part="R4" gate="G$1" pin="1"/>
 </segment>
@@
 </segment>
 </net>
+<net name="N$4" class="0">
+<segment>
+<pinref part="R4" gate="G$1" pin="2"/>
+<pinref part="T1" gate="G$1" pin="B"/>
+</segment>
+</net>
 <net name="N$3" class="0">
 <segment>
-<pinref part="T1" gate="G$1" pin="B"/>
-<pinref part="R4" gate="G$1" pin="2"/>
-</segment>
-</net>
+<pinref part="T1" gate="G$1" pin="C"/>
+<pinref part="R2" gate="G$1" pin="1"/>
+<wire x1="-17.78" y1="43.18" x2="-17.78" y2="45.72" width="0.1524" layer="91"/>
+</segment>
+</net>
